Commit message: scara ist ein absoluter Blödsinn

File: environment/machine.xacro (robot description, xacro)
@@ -3,7 +3,7 @@
   <link name="machine_link">
     <visual>
-      <origin xyz="0 0 0" rpy="0 0 0"/>
+      <origin xyz="0 0 0" rpy="1 0 0"/>
       <geometry>
-        <mesh filename="$(find environment)/meshes/machine.stl" scale="10 10 10"/>
+        <mesh filename="$(find environment)/meshes/machine.stl" scale="1 1 1"/>
       </geometry>
     </visual>
@@ -24,5 +24,5 @@
     <parent link="base_link"/>
     <child link="machine_link"/>
-    <origin xyz="1 0 0" rpy="0 0 0"/>
+    <origin xyz="0 0 0" rpy="0 0 0"/>
   </joint>
 </robot>

File: scara/urdf/scara.xacro (robot description, xacro)
@@ -140,8 +140,8 @@
       xyz="0 0 1" />
     <limit
-      lower="0"
-      upper="0"
-      effort="0"
-      velocity="0" />
+      lower="-1.57"
+      upper="1.57"
+      effort="5"
+      velocity="1.5" />
   </joint>
   <link name="${prefix}M3">
@@ -194,8 +194,8 @@
       xyz="0 0 -1" />
     <limit
-      lower="0"
-      upper="0"
-      effort="0"
-      velocity="0" />
+      lower="1.57"
+      upper="1.57"
+      effort="5"
+      velocity="1.5" />
   </joint>
   <link name="${prefix}M4R">
@@ -298,7 +298,7 @@
     <limit
       lower="0"
-      upper="0"
-      effort="0"
-      velocity="0" />
+      upper="0.4"
+      effort="5"
+      velocity="1.5" />
   </joint>
 </robot>
