Commit message: ready for python

File: polishing_station/description/machine_robots.urdf (robot description, URDF)
Before this commit: robot station_robots, 20 links, 19 joints
Links:
- added link world
- link base_link: mass None -> 10.0
Joints:
- added joint base_to_world: type fixed, parent world, child base_link, origin xyz=0 0 0.01 rpy=0 0 0
- joint frame_to_base_link: origin xyz=0 0 0 rpy=1.57 0 0 -> xyz=0 1.2 0 rpy=1.57 0 0
- joint handler_J1: limit lower=0 upper=0 effort=0 velocity=0 -> lower=-3.141 upper=3.141 effort=5 velocity=1; parent base_link -> handler_base_link
- joint handler_J2: limit lower=0 upper=0 effort=0 velocity=0 -> lower=-3.141 upper=3.141 effort=5 velocity=1
- joint handler_J3: limit lower=0 upper=0 effort=0 velocity=0 -> lower=-3.141 upper=3.141 effort=5 velocity=1
- joint handler_J4: limit lower=0 upper=0 effort=0 velocity=0 -> lower=-3.141 upper=3.141 effort=5 velocity=1
- joint handler_J5: limit lower=0 upper=0 effort=0 velocity=0 -> lower=-3.141 upper=3.141 effort=5 velocity=1
- joint handler_J6: limit lower=0 upper=0 effort=0 velocity=0 -> lower=-3.141 upper=3.141 effort=5 velocity=1
- joint handler_base_to_base_link: origin xyz=0 3 0 rpy=0 0 0 -> xyz=0.9635 0.9 0.27 rpy=0 0 0
- joint polisher_J1: parent base_link -> polisher_base_link
- joint polisher_base_to_base_link: origin xyz=3 3 0 rpy=0 0 0 -> xyz=0.6 0.6 1.95 rpy=3.141 0 0
- joint scara_J1: parent base_link -> scara_base_link
- joint scara_base_to_base_link: origin xyz=3 0 0 rpy=0 0 0 -> xyz=0.6 0.14 0.67 rpy=0 0 0

File: polishing_station/description/machine_robots.xacro (robot description, xacro)
@@ -6,4 +6,9 @@
   name="station_robots">
 <link name="base_link"/>
+<joint name="frame_to_base_link" type="fixed">
+    <parent link="base_link"/>
+    <child link="static_frame"/>
+    <origin xyz="0 1.2 0" rpy="1.57 0 0"/>
+</joint>
 <joint name="scara_base_to_base_link" type="fixed">
     <origin xyz="3 0 0" rpy="0 0 0"/>
@@ -12,5 +17,5 @@
 </joint>
 <joint name="handler_base_to_base_link" type="fixed">
-    <origin xyz="0 3 0" rpy="0 0 0"/> <!-- adjust xyz if needed -->
+    <origin xyz="0.963 0.27 0.9" rpy="0 0 0"/> <!-- adjust xyz if needed -->
     <parent link="base_link"/>
     <child link="handler_base_link"/>
@@ -20,9 +25,4 @@
     <parent link="base_link"/>
     <child link="polisher_base_link"/>
-</joint>
-<joint name="frame_to_base_link" type="fixed">
-    <parent link="base_link"/>
-    <child link="static_frame"/>
-    <origin xyz="0 0 0" rpy="1.57 0 0"/>
 </joint>
 <link name="static_frame">
@@ -413,8 +413,8 @@
       xyz="0 1 0" />
     <limit
-      lower="0"
-      upper="0"
-      effort="0"
-      velocity="0" />
+      lower="-3.141"
+      upper="3.141"
+      effort="5"
+      velocity="1" />
     <dynamics
       damping="1"
@@ -474,8 +474,8 @@
       xyz="1 0 0" />
     <limit
-      lower="0"
-      upper="0"
-      effort="0"
-      velocity="0" />
+      lower="-3.141"
+      upper="3.141"
+      effort="5"
+      velocity="1" />
     <dynamics
       damping="1"
@@ -535,8 +535,8 @@
       xyz="1 0 0" />
     <limit
-      lower="0"
-      upper="0"
-      effort="0"
-      velocity="0" />
+      lower="-3.141"
+      upper="3.141"
+      effort="5"
+      velocity="1" />
     <dynamics
       damping="1"
@@ -596,8 +596,8 @@
       xyz="1 0 0" />
     <limit
-      lower="0"
-      upper="0"
-      effort="0"
-      velocity="0" />
+      lower="-3.141"
+      upper="3.141"
+      effort="5"
+      velocity="1" />
     <dynamics
       damping="1"
@@ -657,8 +657,8 @@
       xyz="0 0 1" />
     <limit
-      lower="0"
-      upper="0"
-      effort="0"
-      velocity="0" />
+      lower="-3.141"
+      upper="3.141"
+      effort="5"
+      velocity="1" />
     <dynamics
       damping="1"
@@ -718,8 +718,8 @@
       xyz="0 1 0" />
     <limit
-      lower="0"
-      upper="0"
-      effort="0"
-      velocity="0" />
+      lower="-3.141"
+      upper="3.141"
+      effort="5"
+      velocity="1" />
     <dynamics
       damping="1"

Commit message: cant find the reason base_link isnt published via /tf

File: polishing_station/description/machine_robots.urdf (robot description, URDF)
Before this commit: robot station_robots, 21 links, 20 joints
Joints:
- joint base_to_world: origin xyz=0 0 0.01 rpy=0 0 0 -> xyz=0 0 1 rpy=0 0 0
- joint scara_base_to_base_link: origin xyz=0.6 0.14 0.67 rpy=0 0 0 -> xyz=0.6 0.14 0.75 rpy=0 0 0

Commit message: idk used j states instead of positions

File: polishing_station/description/machine_robots.urdf (robot description, URDF)
Before this commit: robot station_robots, 21 links, 20 joints
Joints:
- joint base_to_world: origin xyz=0 0 1 rpy=0 0 0 -> xyz=0 0 0.01 rpy=0 0 0
- joint scara_base_to_base_link: origin xyz=0.6 0.14 0.75 rpy=0 0 0 -> xyz=0.6 0.14 0.67 rpy=0 0 0

Commit message: working on attaching

File: polishing_station/description/machine_robots.urdf (robot description, URDF)
Before this commit: robot station_robots, 21 links, 20 joints
Links:
- added link vacuum_gripper_handler, mass 0.001; collision cylinder length=0.01 radius=0.005; visual cylinder length=0.01 radius=0.005
- added link vacuum_gripper_scara, mass 0.001; collision cylinder length=0.02 radius=0.05; visual cylinder length=0.01 radius=0.005
Joints:
- added joint vacuum_gripper_handler_joint: type fixed, parent handler_L6, child vacuum_gripper_handler, origin xyz=0 0.04 0 rpy=1.571 0 0
- added joint vacuum_gripper_scara_joint: type fixed, parent scara_L4, child vacuum_gripper_scara, origin xyz=0.0 0.10 0.0 rpy=1.571 0 0
- joint scara_J4: limit lower=-0.12 upper=0 effort=5 velocity=1 -> lower=-0.14 upper=0 effort=5 velocity=1

File: polishing_station/handler/urdf/handler.urdf (robot description, URDF)
Before this commit: robot handler, 7 links, 6 joints
Links:
- added link vacuum_gripper_handler; visual cylinder length=0.05 radius=0.02
Joints:
- added joint vacuum_gripper_handler_joint: type fixed, parent L6, child vacuum_gripper_handler, origin xyz=0 0 0.05 rpy=0 0 0

File: polishing_station/scara/urdf/scara.urdf (robot description, URDF)
Before this commit: robot scara, 5 links, 4 joints
Links:
- added link vacuum_gripper_scara; visual cylinder length=0.05 radius=0.02
Joints:
- added joint vacuum_gripper_scara_joint: type fixed, parent L4, child vacuum_gripper_scara, origin xyz=0 0 0.05 rpy=0 0 0

Commit message: further progress in attaching detaching workflow

File: polishing_station/description/machine_robots.urdf (robot description, URDF)
Before this commit: robot station_robots, 23 links, 22 joints
Links:
- removed link vacuum_gripper_handler
- removed link vacuum_gripper_scara
Joints:
- removed joint vacuum_gripper_handler_joint
- removed joint vacuum_gripper_scara_joint
- joint scara_J4: limit lower=-0.14 upper=0 effort=5 velocity=1 -> lower=-0.16 upper=0.1 effort=5 velocity=1

File: polishing_station/description/phone.urdf (robot description, URDF)
Before this commit: robot phone, 1 links, 0 joints
Links:
- link phone_link: mass 1.0 -> 0.15; geometry collision box size=0.05 0.07 0.01; visual mesh filename=package://polishing_station/objects/meshes/phone.stl scale=1 1 1
